File: msp430_Keyboard.kicad_pcb (KiCad board)
At the start: 2 copper layers, 285.2 x 94.9 mm, 180 parts, among them J1 Conn_01x04_Male, J2 USB_C_Receptacle_USB2.0, J3 Conn_01x02_Male, SW1 `, SW10 2, SW11 W, SW12 S, SW13 Y, SW14 L_Super, SW15 3, SW16 E, SW17 D, SW18 X, SW19 4, SW2 TAB, SW20 R, SW21 F, SW22 C, SW23 5, SW24 T, SW25 G, SW26 V, SW27 6, SW28 Z, SW29 H, SW3 ESC, SW30 B, SW31 Space, SW32 7, SW33 U, SW34 J, SW35 N, SW36 8, SW37 I, SW38 K, SW39 M, SW4 L_Ctrl, SW40 9, SW41 O, SW42 L, SW43 ,, SW44 0, SW45 P, SW46 ;, SW47 ., SW48 R_Ctrl, SW49 -, SW5 L_Shift, SW50 [, SW51 ', SW52 /, SW53 R_Shift, SW54 =, SW55 ], SW56 \, SW57 Alt_GR, SW58 Backspace, SW59 Enter, SW6 1, SW60 R_Super, SW61 FUNC, SW62 SW_Push, SW63 SW_Push, SW64 Rotary_Encoder_Switch, SW7 Q, SW8 A, SW9 L_Alt, U1 MSP430F5510IRGZ, U2 74LS138, U3 74LS138, U4 Micro-32-HS-Wismar, U5 MCP73831-2-OT, U6 AMS1117-3.3, Y1 12MHz, Y2 32.768kHz

Commit message: Layout fortgesetzt
Parts:
- added D55: LED_Small, LED_THT:LED_D3.0mm_Horizontal_O1.27mm_Z2.0mm, F.Cu at (203.6, 81.5)
- added R11: 470, Resistor_SMD:R_0603_1608Metric_Pad0.98x0.95mm_HandSolder, B.Cu at (205.1, 79.5)
- moved U3 87.6 mm to (83.8, 76.5), turned to 90 degrees
- moved C2 80.9 mm to (86.1, 71.2), turned to 90 degrees
- moved C1 14.3 mm to (80.3, 71.2), turned to 90 degrees
- moved U2 6.86 mm to (78.0, 76.5), turned to 90 degrees
- moved R9 0.89 mm to (107.6, 10.9)
- moved U5 0.89 mm to (107.6, 13.3)
- moved C7 0.28 mm to (110.4, 13.3)
- moved C6 0.25 mm to (104.5, 13.3)
Connections:
- U4 pad 24: Net-(SW63-Pad1) -> Net-(U4-Pad24)
- U4 pad 25: Net-(U4-Pad25) -> Net-(SW63-Pad1)
Routing:
- net /Switch_Matrix/B: track 0.00 -> 227.7 mm, vias 0 -> 4
- net /Switch_Matrix/A: track 0.00 -> 227.2 mm, vias 0 -> 4
- net Net-(D51-Pad1): track 0.00 -> 160.9 mm, vias 0 -> 3
- net /USB/D+: track 7.88 -> 143.5 mm, vias 1 -> 5
- net /USB/D-: track 4.65 -> 139.9 mm, vias 1 -> 4
- net VBUS: track 2.54 -> 134.8 mm, vias 0 -> 4
- net Net-(R10-Pad1): track 0.00 -> 118.7 mm, vias 0 -> 1
- net Net-(D12-Pad1): track 0.00 -> 80.9 mm, vias 0 -> 4
- net Net-(D4-Pad1): track 0.00 -> 80.9 mm, vias 0 -> 4
- net Net-(D16-Pad1): track 0.00 -> 78.7 mm, vias 0 -> 4
- net Net-(D28-Pad1): track 0.00 -> 78.2 mm, vias 0 -> 4
- net Net-(D10-Pad1): track 0.00 -> 78.2 mm, vias 0 -> 4
- net Net-(D20-Pad1): track 0.00 -> 77.9 mm, vias 0 -> 4
- net Net-(D40-Pad1): track 0.00 -> 77.7 mm, vias 0 -> 4
- net Net-(D36-Pad1): track 0.00 -> 77.7 mm, vias 0 -> 4
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
Commit message: Layout sent to JLCPCB
Parts:
- added C19: 1n, Capacitor_SMD:C_0603_1608Metric_Pad1.08x0.95mm_HandSolder, B.Cu at (110.7, 73.4)
- added R12: 47k, Resistor_SMD:R_0603_1608Metric_Pad0.98x0.95mm_HandSolder, B.Cu at (107.7, 73.4)
- added REF**: OSHW-Logo2_14.6x12mm_SilkScreen, HS-Wismar:OSHW-Logo2_14.6x12mm_SilkScreen, B.Cu at (268.1, 56.1)
- added SW65: SW_SPDT, HS-Wismar:APEM_SLG12014, B.Cu at (20.2, 38.1)
- C1, C2: footprint Capacitor_SMD:C_0603_1608Metric -> Capacitor_SMD:C_0603_1608Metric_Pad1.08x0.95mm_HandSolder
- C10, C11, C12, C13, C14, C15, C16, C17, C18, JP1: moved to B.Cu
- C3, C4: value C_Small -> 15p; footprint Capacitor_SMD:C_0603_1608Metric -> Capacitor_SMD:C_0603_1608Metric_Pad1.08x0.95mm_HandSolder; moved to F.Cu
- C5: value C_Small -> 10u; footprint Capacitor_SMD:C_0603_1608Metric -> Capacitor_SMD:C_1206_3216Metric_Pad1.33x1.80mm_HandSolder; moved to B.Cu
- R1, R2, R3, R4, R5, R6, R7, R8: footprint Resistor_SMD:R_0603_1608Metric -> Resistor_SMD:R_0603_1608Metric_Pad0.98x0.95mm_HandSolder
- U1, U2, U3, Y1: moved to F.Cu
- moved U3 146.1 mm to (228.6, 57.0)
- moved C2 141.1 mm to (226.3, 55.1), turned to 270 degrees
- moved R1 100.5 mm to (29.5, 6.48), turned to 90 degrees
- moved R2 79.6 mm to (38.6, 25.5), turned to 90 degrees
- moved R3 68.3 mm to (43.3, 44.6), turned to 90 degrees
- moved C1 51.2 mm to (30.9, 57.8), turned to 0 degrees
- moved R4 50.0 mm to (53.2, 63.6), turned to 90 degrees
- moved U2 48.7 mm to (31.4, 62.4)
- moved Y2 30.7 mm to (71.2, 76.5), turned to 90 degrees
- moved C4 25.4 mm to (76.5, 71.2), turned to 180 degrees
- moved C8 24.2 mm to (77.1, 32.3)
- moved C9 23.9 mm to (65.5, 32.1)
- moved U6 23.9 mm to (71.4, 32.3)
- moved C14 22.2 mm to (72.8, 78.6), turned to 180 degrees
- moved C11 22.1 mm to (73.5, 74.8), turned to 180 degrees
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Connections:
- C8 pad 1: +BATT -> Net-(C8-Pad1)
- U1 pad 22: Net-(U1-Pad22) -> Net-(SW61-Pad1)
- U1 pad 5: Net-(SW61-Pad1) -> Net-(U1-Pad5)
- U6 pad 3: +BATT -> Net-(C8-Pad1)
Routing:
- net +3V3: track 10.2 -> 366.3 mm, vias 0 -> 10
- net Net-(SW53-Pad1): track 0.00 -> 206.4 mm, vias 0 -> 1
- net /Switch_Matrix/Col_1: track 17.5 -> 223.7 mm, vias 2 -> 5
- net /Switch_Matrix/Col_0: track 17.7 -> 223.8 mm, vias 2 -> 5
- net /Switch_Matrix/Col_2: track 18.7 -> 224.4 mm, vias 2 -> 5
- net /Switch_Matrix/Col_3: track 20.2 -> 221.7 mm, vias 2 -> 5
- net Net-(SW61-Pad1): track 0.00 -> 196.7 mm, vias 0 -> 1
- net Net-(SW48-Pad1): track 0.00 -> 182.0 mm, vias 0 -> 1
- net Net-(SW60-Pad1): track 0.00 -> 152.6 mm, vias 0 -> 1
- net Net-(SW57-Pad1): track 0.00 -> 126.5 mm, vias 0 -> 1
- net Net-(D28-Pad1): track 78.2 -> 191.8 mm, vias 4 -> 6
- net /Switch_Matrix/Row_0: track 0.00 -> 103.7 mm, vias 0 -> 1
- net Net-(SW5-Pad1): track 0.00 -> 95.8 mm, vias 0 -> 3
- net Net-(D24-Pad1): track 77.2 -> 167.2 mm, vias 4 -> 6
- net /esp32/EN_\RST: track 0.00 -> 84.4 mm, vias 0 -> 3
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Other:
- board text added: "MSP430_KeyB - A.Wenzel - 26.07.2021"

Commit message: Filterung in den USB-Leitungen, VBus besser abgeblockt, Enter Taste gedreht
Parts:
- added C20: 1μ, Capacitor_SMD:C_0603_1608Metric_Pad1.08x0.95mm_HandSolder, B.Cu at (81.2, 67.1)
- added C21: 10μ, Capacitor_SMD:C_1206_3216Metric_Pad1.33x1.80mm_HandSolder, F.Cu at (9.40, 4.45)
- added C22: 10p, Capacitor_SMD:C_0603_1608Metric_Pad1.08x0.95mm_HandSolder, B.Cu at (10.3, 6.48)
- added C23: 10p, Capacitor_SMD:C_0603_1608Metric_Pad1.08x0.95mm_HandSolder, B.Cu at (13.6, 6.48)
- added R13: 1Meg, Resistor_SMD:R_0603_1608Metric_Pad0.98x0.95mm_HandSolder, B.Cu at (85.7, 72.4)
- added R14: 27, Resistor_SMD:R_0603_1608Metric_Pad0.98x0.95mm_HandSolder, B.Cu at (12.7, 4.06)
- added R15: 27, Resistor_SMD:R_0603_1608Metric_Pad0.98x0.95mm_HandSolder, B.Cu at (11.2, 4.06)
- C5: value 10u -> 10μ
- moved D53 20.8 mm to (259.1, 7.37)
- moved D52 9.60 mm to (262.0, 21.0)
- moved R5 1.57 mm to (85.7, 71.0)
- moved SW65 0.63 mm to (19.8, 38.6)
- turned SW59 to 270 degrees
Connections:
- D53 pad 1: Net-(D48-Pad1) -> Net-(D51-Pad1)
- J2 pad A6: /USB/D+ -> Net-(J2-PadA6)
- J2 pad A7: /USB/D- -> Net-(J2-PadA7)
- J2 pad B6: /USB/D+ -> Net-(J2-PadA6)
- J2 pad B7: /USB/D- -> Net-(J2-PadA7)
Routing:
- net Net-(D53-Pad2): track 37.3 -> 15.6 mm
- net Net-(D51-Pad1): track 91.8 -> 75.8 mm, vias 3 -> 1
- net Net-(R3-Pad1): track 301.9 -> 314.4 mm
- net /USB/D-: track 137.5 -> 126.8 mm, vias 4 -> 3
- net /USB/D+: track 139.9 -> 129.9 mm, vias 5 -> 4
- net Net-(J2-PadA6): track 0.00 -> 9.21 mm, vias 0 -> 1
- net Net-(J2-PadA7): track 0.00 -> 8.96 mm, vias 0 -> 1
- net VBUS: track 216.4 -> 221.4 mm
- net /Switch_Matrix/A: track 246.1 -> 242.7 mm
- net Net-(D52-Pad2): track 5.79 -> 3.61 mm
- net /Switch_Matrix/B: track 246.7 -> 244.7 mm
- net Net-(R13-Pad2): track 3.49 -> 5.40 mm
- net Net-(C8-Pad1): track 62.6 -> 60.9 mm
- net Net-(R1-Pad1): track 284.4 -> 285.6 mm
- net Net-(D48-Pad1): track 90.1 -> 89.1 mm
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